Commit message: Add realsense_d435i_tilt.urdf.xacro

File: xarm_description/urdf/xarm_device.urdf.xacro (robot description, xacro)
@@ -18,4 +18,5 @@
   <xacro:arg name="ros2_control_params" default=""/>
   <xacro:arg name="add_realsense_d435i" default="false"/>
+  <xacro:arg name="add_realsense_d435i_tilt" default="false"/>
   <xacro:arg name="add_d435i_links" default="true"/>
   <xacro:arg name="use_gazebo_camera" default="false"/>
@@ -48,4 +49,5 @@
     load_gazebo_plugin="true" ros2_control_params="$(arg ros2_control_params)"
     add_realsense_d435i="$(arg add_realsense_d435i)"
+    add_realsense_d435i_tilt="$(arg add_realsense_d435i_tilt)"
     add_d435i_links="$(arg add_d435i_links)"
     add_other_geometry="$(arg add_other_geometry)"

File: xarm_description/urdf/xarm_device_macro.xacro (robot description, xacro)
@@ -20,4 +20,5 @@
     load_gazebo_plugin:=false
     add_realsense_d435i:=false
+    add_realsense_d435i_tilt:=false
     add_d435i_links:=true
     use_gazebo_camera:=false
@@ -200,7 +201,14 @@
       </xacro:unless>
     </xacro:unless>
-    <xacro:if value="${add_realsense_d435i}">
+    <xacro:property name="gripper_fix_attach_xyz" value="0 0 0" />
+    <xacro:if value="${add_realsense_d435i or add_realsense_d435i_tilt}">
       <!-- (xarm) Load RealSense D435i URDF -->
-      <xacro:include filename="$(find xarm_description)/urdf/camera/realsense_d435i.urdf.xacro" />
+      <xacro:if value="${add_realsense_d435i_tilt}">
+        <xacro:include filename="$(find xarm_description)/urdf/camera/realsense_d435i_tilt.urdf.xacro" />
+        <xacro:property name="gripper_fix_attach_xyz" value="0 0 0.005" />
+      </xacro:if>
+      <xacro:unless value="${add_realsense_d435i_tilt}">
+        <xacro:include filename="$(find xarm_description)/urdf/camera/realsense_d435i.urdf.xacro" />
+      </xacro:unless>
       <xacro:d435i_urdf prefix="${prefix}" add_d435i_links="${add_d435i_links}" />
       <xacro:if value="${add_d435i_links}">
@@ -209,5 +217,5 @@
       </xacro:if>
     </xacro:if>
-    <xacro:unless value="${add_realsense_d435i}">
+    <xacro:unless value="${add_realsense_d435i or add_realsense_d435i_tilt}">
       <link name="${prefix}link_eef"/>
     </xacro:unless>
@@ -226,5 +234,6 @@
         <!-- Load XArm Gripper Model URDF -->
         <xacro:include filename="$(find xarm_description)/urdf/gripper/xarm_gripper_macro.xacro" />
-        <xacro:xarm_gripper_macro prefix="${prefix}" attach_to="${prefix}link_eef"
+        <xacro:xarm_gripper_macro prefix="${prefix}"
+          attach_to="${prefix}link_eef" attach_xyz="${gripper_fix_attach_xyz}"
           ros2_control_plugin="${ros2_control_plugin}" dof="${dof}" hard_interface="${hard_interface}" />
       </xacro:unless>
