Commit message: Add load_gazebo_plugin condition to all gazebo elements
* Skip loading transmission.xacro when load_gazebo_plugin is false

File: xarm_description/urdf/gripper/xarm_gripper_macro.xacro (robot description, xacro)
@@ -4,33 +4,49 @@
   <xacro:include filename="$(find xarm_description)/urdf/gripper/xarm_gripper.ros2_control.xacro" />
   <xacro:include filename="$(find xarm_description)/urdf/gripper/xarm_gripper.urdf.xacro" />
-  <xacro:include filename="$(find xarm_description)/urdf/gripper/xarm_gripper.transmission.xacro" />
-  <xacro:include filename="$(find xarm_description)/urdf/gripper/xarm_gripper.gazebo.xacro" />
-  <xacro:macro name="xarm_gripper_macro" params="prefix:='' attach_to:='' ns:='xarm' attach_xyz:='0 0 0' attach_rpy:='0 0 0'
-    ros2_control_plugin:='uf_robot_hardware/UFRobotFakeSystemHardware' dof:=7 hard_interface:='PositionJointInterface' ">
+  <!-- gazebo mimic joint plugin -->
+  <xacro:if value="${load_gazebo_plugin}">
+    <xacro:include filename="$(find xarm_description)/urdf/gripper/xarm_gripper.transmission.xacro" />
+    <xacro:include filename="$(find xarm_description)/urdf/gripper/xarm_gripper.gazebo.xacro" />
+  </xacro:if>
+  <xacro:macro name="xarm_gripper_macro" params="
+    prefix:=''
+    hw_ns:='xarm'
+    attach_to:=''
+    attach_xyz:='0 0 0'
+    attach_rpy:='0 0 0'
+    ros2_control_plugin:='uf_robot_hardware/UFRobotFakeSystemHardware'
+    load_gazebo_plugin:=false
+    dof:=7
+    hard_interface:='PositionJointInterface' "
+    >
     <xacro:if value="${is_ros2 and ros2_control_plugin != 'uf_robot_hardware/UFRobotSystemHardware'}">
       <xacro:xarm_gripper_ros2_control prefix="${prefix}" ros2_control_plugin="${ros2_control_plugin}" />
     </xacro:if>
     <xacro:xarm_gripper_urdf prefix="${prefix}" attach_to="${attach_to}" attach_xyz="${attach_xyz}" attach_rpy="${attach_rpy}" />
-    <xacro:xarm_gripper_transmission prefix="${prefix}" hard_interface="${hard_interface}" />
-    <xacro:xarm_gripper_gazebo prefix="${prefix}" />
-    <xacro:if value="${not is_ros2}">
+    <xacro:if value="${load_gazebo_plugin}">
+      <xacro:xarm_gripper_transmission prefix="${prefix}" hard_interface="${hard_interface}" />
+      <xacro:xarm_gripper_gazebo prefix="${prefix}"/>
+    </xacro:if>
+    <xacro:if value="${load_gazebo_plugin and not is_ros2}">
       <xacro:xarm_gazebo_grasp_fix prefix="${prefix}" palm_link="${prefix}link${dof}" />
     </xacro:if>
     <!-- mimic_joint_plugin has to be installed: -->
-    <xacro:mimic_joint_plugin_gazebo name_prefix="${prefix}left_finger_joint"
-      following_joint="${prefix}drive_joint" mimic_joint="${prefix}left_finger_joint"
-      has_pid="${is_ros2}" multiplier="1.0" max_effort="10.0" />
-    <xacro:mimic_joint_plugin_gazebo name_prefix="${prefix}left_inner_knuckle_joint"
-      following_joint="${prefix}drive_joint" mimic_joint="${prefix}left_inner_knuckle_joint"
-      has_pid="${is_ros2}" multiplier="1.0" max_effort="10.0" />
-    <xacro:mimic_joint_plugin_gazebo name_prefix="${prefix}right_outer_knuckle_joint"
-      following_joint="${prefix}drive_joint" mimic_joint="${prefix}right_outer_knuckle_joint"
-      has_pid="${is_ros2}" multiplier="1.0" max_effort="10.0" />
-    <xacro:mimic_joint_plugin_gazebo name_prefix="${prefix}right_finger_joint"
-      following_joint="${prefix}drive_joint" mimic_joint="${prefix}right_finger_joint"
-      has_pid="${is_ros2}" multiplier="1.0" max_effort="10.0" />
-    <xacro:mimic_joint_plugin_gazebo name_prefix="${prefix}right_inner_knuckle_joint"
-      following_joint="${prefix}drive_joint" mimic_joint="${prefix}right_inner_knuckle_joint"
-      has_pid="${is_ros2}" multiplier="1.0" max_effort="10.0" />
+    <xacro:if value="${load_gazebo_plugin}">
+      <xacro:mimic_joint_plugin_gazebo name_prefix="${prefix}left_finger_joint"
+        following_joint="${prefix}drive_joint" mimic_joint="${prefix}left_finger_joint"
+        has_pid="${is_ros2}" multiplier="1.0" max_effort="10.0" />
+      <xacro:mimic_joint_plugin_gazebo name_prefix="${prefix}left_inner_knuckle_joint"
+        following_joint="${prefix}drive_joint" mimic_joint="${prefix}left_inner_knuckle_joint"
+        has_pid="${is_ros2}" multiplier="1.0" max_effort="10.0" />
+      <xacro:mimic_joint_plugin_gazebo name_prefix="${prefix}right_outer_knuckle_joint"
+        following_joint="${prefix}drive_joint" mimic_joint="${prefix}right_outer_knuckle_joint"
+        has_pid="${is_ros2}" multiplier="1.0" max_effort="10.0" />
+      <xacro:mimic_joint_plugin_gazebo name_prefix="${prefix}right_finger_joint"
+        following_joint="${prefix}drive_joint" mimic_joint="${prefix}right_finger_joint"
+        has_pid="${is_ros2}" multiplier="1.0" max_effort="10.0" />
+      <xacro:mimic_joint_plugin_gazebo name_prefix="${prefix}right_inner_knuckle_joint"
+        following_joint="${prefix}drive_joint" mimic_joint="${prefix}right_inner_knuckle_joint"
+        has_pid="${is_ros2}" multiplier="1.0" max_effort="10.0" />
+    </xacro:if>
   </xacro:macro>
 </robot>

File: xarm_description/urdf/xarm7/xarm7_robot_macro.xacro (robot description, xacro)
@@ -9,4 +9,5 @@
     add_bio_gripper:=false
     ros2_control_plugin:='uf_robot_hardware/UFRobotSystemHardware'
+    load_gazebo_plugin:=false
     robot_ip:=''
     report_type:='normal'
@@ -23,6 +24,8 @@
     </xacro:if>
     <xacro:include filename="$(find xarm_description)/urdf/xarm7/xarm7.urdf.xacro" />
-    <xacro:include filename="$(find xarm_description)/urdf/xarm7/xarm7.transmission.xacro" />
-    <xacro:include filename="$(find xarm_description)/urdf/xarm7/xarm7.gazebo.xacro" />
+    <xacro:if value="${load_gazebo_plugin}">
+      <xacro:include filename="$(find xarm_description)/urdf/xarm7/xarm7.transmission.xacro" />
+      <xacro:include filename="$(find xarm_description)/urdf/xarm7/xarm7.gazebo.xacro" />
+    </xacro:if>
     <xacro:if value="${limited}">
       <xacro:if value="${is_ros2}">
@@ -67,6 +70,8 @@
         />
     </xacro:unless>
-    <xacro:xarm7_transmission prefix="${prefix}" hard_interface="${hard_interface}" />
-    <xacro:xarm7_gazebo prefix="${prefix}" />
+    <xacro:if value="${load_gazebo_plugin}">
+      <xacro:xarm7_transmission prefix="${prefix}" hard_interface="${hard_interface}" />
+      <xacro:xarm7_gazebo prefix="${prefix}" />
+    </xacro:if>
   </xacro:macro>
 </robot>

File: xarm_description/urdf/xarm_device.urdf.xacro (robot description, xacro)
@@ -17,4 +17,5 @@
   <xacro:arg name="ros2_control_plugin" default="uf_robot_hardware/UFRobotSystemHardware"/>
   <xacro:arg name="ros2_control_params" default=""/>
+  <xacro:arg name="load_gazebo_plugin" default="true"/>
   <xacro:arg name="add_realsense_d435i" default="false"/>
   <xacro:arg name="add_realsense_d435i_tilt" default="false"/>
@@ -47,5 +48,5 @@
     add_bio_gripper="$(arg add_bio_gripper)" dof="$(arg dof)"
     ros2_control_plugin="$(arg ros2_control_plugin)" robot_type="$(arg robot_type)"
-    load_gazebo_plugin="true" ros2_control_params="$(arg ros2_control_params)"
+    load_gazebo_plugin="$(arg load_gazebo_plugin)" ros2_control_params="$(arg ros2_control_params)"
     add_realsense_d435i="$(arg add_realsense_d435i)"
     add_realsense_d435i_tilt="$(arg add_realsense_d435i_tilt)"

File: xarm_description/urdf/xarm_device_macro.xacro (robot description, xacro)
@@ -212,5 +212,5 @@
       </xacro:unless>
       <xacro:d435i_urdf prefix="${prefix}" add_d435i_links="${add_d435i_links}" />
-      <xacro:if value="${add_d435i_links}">
+      <xacro:if value="${load_gazebo_plugin and add_d435i_links}">
         <xacro:include filename="$(find xarm_description)/urdf/camera/realsense.gazebo.xacro" />
         <xacro:realsense_gazebo prefix="${prefix}" />
