Commit message: Reverse xarm gripper joint axes to match with API

File: xarm_description/urdf/gripper/xarm_gripper.urdf.xacro (robot description, xacro)
@@ -46,8 +46,8 @@
     </link>
     <joint name="${prefix}drive_joint" type="revolute">
-      <origin xyz="0 0.035 0.059098" rpy="0 0 0" />
+      <origin xyz="0 0.035 0.059098" rpy="0.85 0 0" />
       <parent link="${prefix}xarm_gripper_base_link" />
       <child link="${prefix}left_outer_knuckle" />
-      <axis xyz="1 0 0" />
+      <axis xyz="-1 0 0" />
       <limit lower="0" upper="0.85" effort="50" velocity="2" />
     </joint>
@@ -71,8 +71,8 @@
     </link>
     <joint name="${prefix}left_finger_joint" type="revolute">
-      <origin xyz="0 0.035465 0.042039" rpy="0 0 0" />
+      <origin xyz="0 0.035465 0.042039" rpy="-0.85 0 0" />
       <parent link="${prefix}left_outer_knuckle" />
       <child link="${prefix}left_finger" />
-      <axis xyz="-1 0 0" />
+      <axis xyz="1 0 0" />
       <limit lower="0" upper="0.85" effort="50" velocity="2" />
       <mimic joint="${prefix}drive_joint" multiplier="1" offset="0" />
@@ -97,8 +97,8 @@
     </link>
     <joint name="${prefix}left_inner_knuckle_joint" type="revolute">
-      <origin xyz="0 0.02 0.074098" rpy="0 0 0" />
+      <origin xyz="0 0.02 0.074098" rpy="0.85 0 0" />
       <parent link="${prefix}xarm_gripper_base_link" />
       <child link="${prefix}left_inner_knuckle" />
-      <axis xyz="1 0 0" />
+      <axis xyz="-1 0 0" />
       <limit lower="0" upper="0.85" effort="50" velocity="2" />
       <mimic joint="${prefix}drive_joint" multiplier="1" offset="0" />
@@ -123,8 +123,8 @@
     </link>
     <joint name="${prefix}right_outer_knuckle_joint" type="revolute">
-      <origin xyz="0 -0.035 0.059098" rpy="0 0 0" />
+      <origin xyz="0 -0.035 0.059098" rpy="-0.85 0 0" />
       <parent link="${prefix}xarm_gripper_base_link" />
       <child link="${prefix}right_outer_knuckle" />
-      <axis xyz="-1 0 0" />
+      <axis xyz="1 0 0" />
       <limit lower="0" upper="0.85" effort="50" velocity="2" />
       <mimic joint="${prefix}drive_joint" multiplier="1" offset="0" />
@@ -149,8 +149,8 @@
     </link>
     <joint name="${prefix}right_finger_joint" type="revolute">
-      <origin xyz="0 -0.035465 0.042039" rpy="0 0 0" />
+      <origin xyz="0 -0.035465 0.042039" rpy="0.85 0 0" />
       <parent link="${prefix}right_outer_knuckle" />
       <child link="${prefix}right_finger" />
-      <axis xyz="1 0 0" />
+      <axis xyz="-1 0 0" />
       <limit lower="0" upper="0.85" effort="50" velocity="2" />
       <mimic joint="${prefix}drive_joint" multiplier="1" offset="0" />
@@ -175,8 +175,8 @@
     </link>
     <joint name="${prefix}right_inner_knuckle_joint" type="revolute">
-      <origin xyz="0 -0.02 0.074098" rpy="0 0 0" />
+      <origin xyz="0 -0.02 0.074098" rpy="-0.85 0 0" />
       <parent link="${prefix}xarm_gripper_base_link" />
       <child link="${prefix}right_inner_knuckle" />
-      <axis xyz="-1 0 0" />
+      <axis xyz="1 0 0" />
       <limit lower="0" upper="0.85" effort="50" velocity="2" />
       <mimic joint="${prefix}drive_joint" multiplier="1" offset="0" />
